File: paws60/pcb/Hotswap/matrix.kicad_sch (KiCad schematic)
At the start: 142 parts

Commit message: Updated PCB for Paws60, remove ISO layout
Parts:
- removed D42, D45: 1N4148, Diode_SMD:D_SOD-123, symbol Device:D
- removed MX44, MX49: 1u, MX_Only:MXOnly-1U-Hotswap, symbol Switch:SW_SPST
- removed MX46: ISO, MX_Only:MXOnly-ISO-ROTATED-Hotswap-ReversedStabilizers-Left, symbol Switch:SW_SPST
- removed MX47: 1.25u, MX_Only:MXOnly-1.25U-Hotswap, symbol Switch:SW_SPST
- MX30: footprint MX_Only:MXOnly-1.5U-Hotswap-Rotated -> MX_Only:MXOnly-1.5U-Hotswap
- MX44: renamed from MX45; footprint MX_Only:MXOnly-2.25U-Hotswap-ReversedStabilizers-Left -> MX_Only:MXOnly-2.25U-Hotswap
- MX58: renamed from MX62; footprint MX_Only:MXOnly-2.75U-Hotswap -> MX_Only:MXOnly-2.75U-Hotswap-ReversedStabilizers
- renumbered D43 to D42, D44 to D43, D46 to D44, D47 to D45, D48 to D46, D49 to D47, D50 to D48, D51 to D49, D52 to D50, D53 to D51, D54 to D52, D55 to D53, D56 to D54, D57 to D55, D58 to D56, D59 to D57, D60 to D58, D61 to D59, D62 to D60, D63 to D61, D64 to D62, D65 to D63, MX48 to MX45, MX50 to MX46, MX51 to MX47, MX52 to MX48, MX53 to MX49, MX54 to MX50, MX55 to MX51, MX56 to MX52, MX57 to MX53, MX58 to MX54, MX59 to MX55, MX60 to MX56, MX61 to MX57, MX63 to MX59, MX64 to MX60, MX65 to MX61, MX66 to MX62, MX67 to MX63, MX68 to MX64, MX69 to MX65, MX70 to MX66, MX71 to MX67, MX72 to MX68, MX73 to MX69, MX74 to MX70, MX75 to MX71, MX76 to MX72, MX77 to MX73

Commit message: Re-wire, ...
Parts:
- MX58: footprint MX_Only:MXOnly-2.75U-Hotswap-ReversedStabilizers -> MX_Only:MXOnly-2.75U-Hotswap
