File: sakura50/pcb/rev1/sakura50.kicad_sch (KiCad schematic)
At the start: 154 parts, among them J1 OLED, J2 AVR-ISP-6, J3 JST SH 4-pin, J4 Battery, SW1 Reset, SW2 Reset, U1 BlueMacro, U2 ATmega32U4-AU, U3 USBLC6-2SC6, Y1 16Mhz

Commit message: Update new layout change for sakura50
Parts:
- removed D38: 1N4148, Diode_SMD:D_SOD-123, symbol Device:D
- removed MX40: 1u, MX_Only:MXOnly-1U-Hotswap, symbol Switch:SW_SPST
- added D46: 1N4148, Diode_SMD:D_SOD-123, symbol Device:D
- added MX48: 1u, MX_Only:MXOnly-1U-Hotswap, symbol Switch:SW_SPST
- added S1, S2: Screw_Side, Type-C:10x5_7x2.5mm, symbol Connector:Screw_Terminal_01x01
- MX39: value 2u -> 2.25u; footprint MX_Only:MXOnly-2U-Hotswap -> MX_Only:MXOnly-2.25U-Hotswap
- MX47: renamed from MX48; value 2u -> 1u; footprint MX_Only:MXOnly-2U-Hotswap -> MX_Only:MXOnly-1U-Hotswap
- MX49: value 1u -> 1.75u; footprint MX_Only:MXOnly-1U-Hotswap -> MX_Only:MXOnly-1.75U-Hotswap
- renumbered D39 to D38, D40 to D39, D41 to D40, D42 to D41, D43 to D42, D44 to D43, D45 to D44, D46 to D45, MX41 to MX40, MX42 to MX41, MX43 to MX42, MX44 to MX43, MX45 to MX44, MX46 to MX45, MX47 to MX46
Connections:
- net GND: now also S1.1 (Pin_1), S2.1 (Pin_1)
- net col1: no longer MX61.2 (B)
- net col10: now also MX57.2 (B), MX63.2 (B), MX48.2 (B)
- net col11: now also MX58.2 (B)
- net col2: now also MX61.2 (B)
- net col3: no longer MX54.2 (B)
- net col4: now also MX54.2 (B)
- net col5: no longer MX55.2 (B), MX62.2 (B)
- net col6: now also MX55.2 (B), MX62.2 (B)
- net col7: no longer MX56.2 (B)
- net col8: now also MX56.2 (B); no longer MX57.2 (B)
- net col9: no longer MX58.2 (B), MX63.2 (B)
- net row3: now also D46.1 (K)
- net at D55.2 (A), MX57.1 (A): now also MX63.1 (A)
- net at D50.2 (A), MX52.1 (A): no longer MX61.1 (A)
- net at D56.2 (A), MX58.1 (A): no longer MX63.1 (A)
- net at D51.2 (A), MX53.1 (A): now also MX61.1 (A)
- new net: D46.2 (A), MX48.1 (A)
Other:
- moved on the sheet: D52, D53, D54, D55, D56, MX54, MX55, MX56, MX57, MX58, MX61, MX62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

Commit message: Added new revision for Sakura50 board
Other:
- title: Sakura60 (Not Final) -> Sakura50
