File: sakura50/pcb/rev2/sakura50.kicad_sch (KiCad schematic)
At the start: 281 parts, among them J1 OLED, J2 ARM-JTAG-6, J3 JST SH 4-pin, J4 Battery, SW1 Reset, SW2 Reset, SW3 Boot0, SW4 Boot1, U1 BlueMacro, U2 STM32F303CCTx, U3 AT24C512C-SSHD-T, Y1 8Mhz

Commit message: Updated some issue fix
Parts:
- added R13, R14, R15, R16, R17: 10k, Resistor_SMD:R_0805_2012Metric, symbol Device:R
- R9: value 10k -> 1.5k
Connections:
- net SCL: now also R14.1
- net SDA: now also R15.1
- net SK6812: now also R13.2
- net VCC: now also R13.1, R14.2, R15.2
- net rot0: now also U2.2 (PC13), R16.1; no longer C2.1, U2.4 (PC15)
- net rot1: now also U2.4 (PC15), R17.1; no longer C3.1, U2.2 (PC13)
- new net: C2.1, R16.2
- new net: C3.1, R17.2
Other:
- moved on the sheet: C2, C3

Commit message: Added LDO XC6206, and re-wire a bit
Parts:
- added C77, C78: 1.0u, Capacitor_SMD:C_0805_2012Metric, symbol Device:C
- added RG1: XC6206P332MR, Torex-XC6206P332MR, symbol eec:XC6206P332MR
Connections:
- net GND: now also C77.1, C78.2, RG1.1 (VSS)
- net VBUS: now also C78.1, RG1.3 (VIN)
- net VCC: now also C77.2, RG1.2 (VOUT)

Commit message: Added rev 2 for Paws60 pcb
Parts:
- removed C22: 100nF, Capacitor_SMD:C_0805_2012Metric, symbol Device:C
- removed LED13: SK6812Mini-e, kbd:YS-SK6812MINI-E, symbol kbd:YS-SK6812MINI-E
- renumbered C23 to C22, C33 to C32, C34 to C33, C35 to C34, C36 to C35, C37 to C36, C38 to C37, C39 to C38, C40 to C39, C41 to C40, C42 to C41, C43 to C42, C44 to C43, C45 to C44, C46 to C45, C47 to C46, C48 to C47, C49 to C48, C50 to C49, C51 to C50, C52 to C51, C53 to C52, C54 to C53, C55 to C54, C56 to C55, C57 to C56, C58 to C57, C59 to C58, C60 to C59, C61 to C60, C62 to C61, C63 to C62, C64 to C63, C65 to C64, C66 to C65, C67 to C66, C68 to C67, C69 to C68, C70 to C69, C71 to C70, C72 to C71, C73 to C72, C74 to C73, C75 to C74, C76 to C75, C32 to C76, LED14 to LED13, LED15 to LED14, LED16 to LED15, LED17 to LED16, LED18 to LED17, LED19 to LED18, LED20 to LED19, LED21 to LED20, LED22 to LED21, LED23 to LED22, LED24 to LED23, LED25 to LED24, LED26 to LED25, LED27 to LED26, LED28 to LED27, LED29 to LED28, LED30 to LED29, LED31 to LED30, LED32 to LED31, LED33 to LED32, LED34 to LED33, LED35 to LED34, LED36 to LED35, LED37 to LED36, LED38 to LED37, LED39 to LED38, LED40 to LED39, LED41 to LED40, LED42 to LED41, LED43 to LED42, LED44 to LED43, LED45 to LED44, LED46 to LED45, LED47 to LED46, LED48 to LED47, LED49 to LED48, LED50 to LED49, LED51 to LED50, LED52 to LED51, LED53 to LED52, LED54 to LED53, LED55 to LED54, LED56 to LED55, LED57 to LED56, LED58 to LED57
Connections:
- net VBUS: now also F1.2; no longer F1.1, J3.1 (Pin_1), R10.1, U1.29 (5V), USB1.11 (VBUS), USB1.2 (VBUS), USB2.4 (VCC)
- net VCC: no longer C10.1, C11.1, C12.1, C13.1, C14.1, C15.1, C16.1, C17.1, C18.1, C19.1, C20.1, C21.1, C22.1, C32.2, C33.2, C34.2, C35.2, C36.2, C37.2, C38.2, C39.2, C40.2, C41.2, C42.2, C43.2, C44.2, C45.2, C46.1, C47.1, C48.1, C49.1, C50.1, C51.1, C52.1, C53.1, C54.1, C55.1, C56.1, C57.1, C58.1, C59.1, C60.2, C61.2, C62.2, C63.2, C64.2, C65.2, C66.2, C67.2, C68.2, C69.2, C70.2, C71.2, C72.2, C73.2, C74.1, C75.1, F1.2, LED1.1 (VDD), LED10.1 (VDD), LED11.1 (VDD), LED12.1 (VDD), LED13.1 (VDD), LED14.1 (VDD), LED15.1 (VDD), LED16.1 (VDD), LED17.1 (VDD), LED18.1 (VDD), LED19.1 (VDD), LED2.1 (VDD), LED20.1 (VDD), LED21.1 (VDD), LED22.1 (VDD), LED23.1 (VDD), LED24.1 (VDD), LED25.1 (VDD), LED26.1 (VDD), LED27.1 (VDD), LED28.1 (VDD), LED29.1 (VDD), LED3.1 (VDD), LED30.1 (VDD), LED31.1 (VDD), LED32.1 (VDD), LED33.1 (VDD), LED34.1 (VDD), LED35.1 (VDD), LED36.1 (VDD), LED37.1 (VDD), LED38.1 (VDD), LED39.1 (VDD), LED4.1 (VDD), LED40.1 (VDD), LED41.1 (VDD), LED42.1 (VDD), LED43.1 (VDD), LED44.1 (VDD), LED45.1 (VDD), LED46.1 (VDD), LED47.1 (VDD), LED48.1 (VDD), LED49.1 (VDD), LED5.1 (VDD), LED50.1 (VDD), LED51.1 (VDD), LED52.1 (VDD), LED53.1 (VDD), LED54.1 (VDD), LED55.1 (VDD), LED56.1 (VDD), LED57.1 (VDD), LED6.1 (VDD), LED7.1 (VDD), LED8.1 (VDD), LED9.1 (VDD), R13.1, R9.1
- net at LED13.4 (DIN): now also LED12.2 (DOUT)
- new net VUSB: C10.1, C11.1, C12.1, C13.1, C14.1, C15.1, C16.1, C17.1, C18.1, C19.1, C20.1, C21.1, C22.1, C32.2, C33.2, C34.2, C35.2, C36.2, C37.2, C38.2, C39.2, C40.2, C41.2, C42.2, C43.2, C44.2, C45.2, C46.1, C47.1, C48.1, C49.1, C50.1, C51.1, C52.1, C53.1, C54.1, C55.1, C56.1, C57.1, C58.1, C59.1, C60.2, C61.2, C62.2, C63.2, C64.2, C65.2, C66.2, C67.2, C68.2, C69.2, C70.2, C71.2, C72.2, C73.2, C74.1, C75.1, F1.1, J3.1 (Pin_1), LED1.1 (VDD), LED10.1 (VDD), LED11.1 (VDD), LED12.1 (VDD), LED13.1 (VDD), LED14.1 (VDD), LED15.1 (VDD), LED16.1 (VDD), LED17.1 (VDD), LED18.1 (VDD), LED19.1 (VDD), LED2.1 (VDD), LED20.1 (VDD), LED21.1 (VDD), LED22.1 (VDD), LED23.1 (VDD), LED24.1 (VDD), LED25.1 (VDD), LED26.1 (VDD), LED27.1 (VDD), LED28.1 (VDD), LED29.1 (VDD), LED3.1 (VDD), LED30.1 (VDD), LED31.1 (VDD), LED32.1 (VDD), LED33.1 (VDD), LED34.1 (VDD), LED35.1 (VDD), LED36.1 (VDD), LED37.1 (VDD), LED38.1 (VDD), LED39.1 (VDD), LED4.1 (VDD), LED40.1 (VDD), LED41.1 (VDD), LED42.1 (VDD), LED43.1 (VDD), LED44.1 (VDD), LED45.1 (VDD), LED46.1 (VDD), LED47.1 (VDD), LED48.1 (VDD), LED49.1 (VDD), LED5.1 (VDD), LED50.1 (VDD), LED51.1 (VDD), LED52.1 (VDD), LED53.1 (VDD), LED54.1 (VDD), LED55.1 (VDD), LED56.1 (VDD), LED57.1 (VDD), LED6.1 (VDD), LED7.1 (VDD), LED8.1 (VDD), LED9.1 (VDD), R10.1, R13.1, R9.1, U1.29 (5V), USB1.11 (VBUS), USB1.2 (VBUS), USB2.4 (VCC)
