File: paws60/pcb/rev2/paws-60-pcb.kicad_sch (KiCad schematic)
At the start: 27 parts, among them J1 JST SH 4-pin, J2 AVR-ISP-6, SW1 Reset, U1 SRV05-4, U2 ATmega32U4-MU, Y1 16MHz

Commit message: Update paws60 hotswap socket footprint and lazulipad
Parts:
- removed S1: Screw_Left, Type-C:10x5_7x2.5mm, symbol Connector:Screw_Terminal_01x01
- removed S2: Screw_Right, Type-C:10x5_7x2.5mm, symbol Connector:Screw_Terminal_01x01
- removed S3, S4, S5, S6: Screw_Plate, Type-C:5.5_5x2.5mm, symbol Connector:Screw_Terminal_01x01
- U: renamed from C1; value 0.1u -> (none); footprint Capacitor_SMD:C_0805_2012Metric -> (none)
- U: renamed from C2; value 0.1u -> (none); footprint Capacitor_SMD:C_0805_2012Metric -> (none)
- U: renamed from C3; value 0.1u -> (none); footprint Capacitor_SMD:C_0805_2012Metric -> (none)
- U: renamed from C4; value 10u -> (none); footprint Capacitor_SMD:C_0805_2012Metric -> (none)
- U: renamed from F1; value 500mA -> (none); footprint Fuse:Fuse_1206_3216Metric -> (none)
- U: renamed from J1; value JST SH 4-pin -> (none); footprint Connector_JST:JST_SH_SM04B-SRSS-TB_1x04-1MP_P1.00mm_Horizontal -> (none)
- U: renamed from R1; value 22 -> (none); footprint Resistor_SMD:R_0805_2012Metric -> (none)
- U: renamed from R2; value 22 -> (none); footprint Resistor_SMD:R_0805_2012Metric -> (none)
- U: renamed from U2; value ATmega32U4-MU -> (none); footprint Package_DFN_QFN:QFN-44-1EP_7x7mm_P0.5mm_EP5.2x5.2mm -> (none)
- U: renamed from SW1; value Reset -> (none); footprint Button_Switch_SMD:SW_SPST_TL3342 -> (none)
- U: renamed from R4; value 10k -> (none); footprint Resistor_SMD:R_0805_2012Metric -> (none)
- U: renamed from C6; value 1u -> (none); footprint Capacitor_SMD:C_0805_2012Metric -> (none)
- U: renamed from R3; value 10k -> (none); footprint Resistor_SMD:R_0805_2012Metric -> (none)
- U: renamed from Y1; value 16MHz -> (none); footprint Crystal:Crystal_SMD_3225-4Pin_3.2x2.5mm -> (none)
- U: renamed from C5; value 22p -> (none); footprint Capacitor_SMD:C_0805_2012Metric -> (none)
- U: renamed from C7; value 22p -> (none); footprint Capacitor_SMD:C_0805_2012Metric -> (none)
- U: renamed from J2; value AVR-ISP-6 -> (none); footprint random-keyboard-parts:Reset_Pretty -> (none)
- U: renamed from U1; value SRV05-4 -> (none); footprint Package_TO_SOT_SMD:SOT-23-6 -> (none)
- U: renamed from LED1; value SK6812Mini-e -> (none); footprint kbd:YS-SK6812MINI-E -> (none)
- U: renamed from R5; value 10k -> (none); footprint Resistor_SMD:R_0805_2012Metric -> (none)
- U: renamed from C8; value 100n -> (none); footprint Capacitor_SMD:C_0805_2012Metric -> (none)
