File: paws60/pcb/rev2/paws60.kicad_sch (KiCad schematic)
At the start: 181 parts

Commit message: Update Paws60 (Rev 2) PCB
Parts:
- added C (x3): C, symbol Device:C
- added LED (x2): SK6812MINI-E, marbastlib-various:LED_6028R, symbol marbastlib-various:SK6812MINI-E
- added U: 74LVC1G17, Package_TO_SOT_SMD:SOT-23-5, symbol kbd:74LVC1G17
Connections:
- net +5V: now also C.1, C.1, C.1, LED.1 (VDD), LED.1 (VDD), U.5 (VCC)
- net GND: now also C.2, C.2, C.2, LED.4 (VSS), LED.4 (VSS), U.3 (GND)
- net ARGB_3V3: now reaches U.35 (GPIO23)
- net ARGB_3V3: now also U.2
- new net: LED.2 (DOUT), LED.3 (DIN)
- new net ARGB_5V: LED.3 (DIN), U.4
- new net VCC: U.5 (VCC)
- no-connect marks 11 -> 10
Other:
- moved on the sheet: C, D, F, J, R, RG, S, SW, U, Y
